Commit message: Update file modified in TP3

File: catkin_ws/src/motoman/motoman_hc10_support/urdf/hc10.xacro (robot description, xacro)
@@ -3,3 +3,9 @@
   <xacro:include filename="$(find motoman_hc10_support)/urdf/hc10_macro.xacro" />
   <xacro:motoman_hc10 prefix=""/>
+  <xacro:include filename="$(find motoman_hc10_support)/urdf/yaskawa.control.xacro"/>
+  <xacro:yaskawa_control arm_id="yaskawa"/>
+  <xacro:include filename="$(find motoman_hc10_support)/urdf/yaskawa.gazebo.xacro"/>
+  <xacro:yaskawa_gazebo arm_id=""/>
+  <xacro:include filename="$(find motoman_hc10_support)/urdf/kinect_camera.gazebo"/>
+  <xacro:camera prefix=""/>
 </robot>

File: catkin_ws/src/motoman/motoman_hc10_support/urdf/hc10_macro.xacro (robot description, xacro)
@@ -199,4 +199,14 @@
       <child link="${prefix}base"/>
     </joint>
+    	<link name="${prefix}camera_rgb_frame"/>
+	<!-- Attach Kinect to table -->
+	<joint type="fixed" name="tool0_camera_joint">
+	    <origin xyz="0.15 -1 0.1" rpy="0 0 1.57"/>
+	    <child link="${prefix}camera_rgb_frame"/>
+	    <parent link="${prefix}tool0"/>
+	    <axis xyz="0 0 0" rpy="0 0 0"/>
+	    <limit effort="10000" velocity="1000"/>
+	    <dynamics damping="1.0" friction="1.0"/>
+	</joint>
   </xacro:macro>
 </robot>

File: catkin_ws/src/motoman/motoman_hc10_support/urdf/test.urdf (robot description, URDF)
Before this commit: robot motoman_hc10, 10 links, 9 joints
Links:
- removed link base
- removed link base_link
- removed link link_1_s
- removed link link_2_l
- removed link link_3_u
- removed link link_4_r
- removed link link_5_b
- removed link link_6_t
- removed link tool0
- removed link world
Joints:
- removed joint base_link-base
- removed joint joint_1_s
- removed joint joint_2_l
- removed joint joint_3_u
- removed joint joint_4_r
- removed joint joint_5_b
- removed joint joint_6_t
- removed joint joint_6_t-tool0
- removed joint world_fixed
